File: hw/blueled.sch (KiCad schematic (older format))
At the start: 56 parts, among them J1 Barrel_Jack, J2 LED Strip, J3 ICSP, J4 Screw_Terminal_01x02, Q1 Q_PMOS_SDG, Q2 Q_PNP_EBC, SW2 PUSH, U1 ATmega328P-AU, U2 HC-05, U3 AMS1117-3.3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

Commit message: add(hw): more components in BOM
Parts:
- L1: Distributor (none) -> lcsc.com; Manuf. Part (none) -> SMMS1040-150M
- R10, R14: footprint (none) -> Resistor_SMD:R_0603_1608Metric_Pad1.05x0.95mm_HandSolder; Manuf. Part RK73B2ATTD102J -> SFR03EZPF1002
- R12: footprint (none) -> Resistor_SMD:R_0603_1608Metric_Pad1.05x0.95mm_HandSolder; Manuf. Part RK73B2ATTD102J -> RC0603FR-072K1L
- R13: footprint (none) -> Resistor_SMD:R_2512_6332Metric_Pad1.52x3.35mm_HandSolder; Manuf. Part RK73B2ATTD102J -> RL2512JK-070R01L
- R9: footprint (none) -> Resistor_SMD:R_0603_1608Metric_Pad1.05x0.95mm_HandSolder; Manuf. Part RK73B2ATTD102J -> MCR03ERTF3401
Changed lines of the file:
@@
 F 1 "15uH" V 5134 1200 50  0000 C CNN
 F 2 "" H 5000 1200 50  0001 C CNN
-F 3 "~" H 5000 1200 50  0001 C CNN
+F 3 "https://datasheet.lcsc.com/szlcsc/1809291526_SXN-Shun-Xiang-Nuo-Elec-SMMS1040-150M_C149596.pdf" H 5000 1200 50  0001 C CNN
+F 4 "lcsc.com" H 5000 1200 50  0001 C CNN "Distributor"
+F 5 "SMMS1040-150M" H 5000 1200 50  0001 C CNN "Manuf. Part"
 	1    5000 1200
 	0    -1   -1   0
@@
 F 0 "R9" H 5709 1946 50  0000 L CNN
 F 1 "3.4k" H 5709 1855 50  0000 L CNN
-F 2 "" H 5650 1900 50  0001 C CNN
-F 3 "" H 5650 1900 50  0001 C CNN
+F 2 "Resistor_SMD:R_0603_1608Metric_Pad1.05x0.95mm_HandSolder" H 5650 1900 50  0001 C CNN
+F 3 "https://datasheet.lcsc.com/szlcsc/ROHM-Semicon-MCR03ERTF3401_C308067.pdf" H 5650 1900 50  0001 C CNN
 F 4 "lcsc.com" H 5650 1900 50  0001 C CNN "Distributor"
-F 5 "RK73B2ATTD102J" H 5650 1900 50  0001 C CNN "Manuf. Part"
+F 5 "MCR03ERTF3401" H 5650 1900 50  0001 C CNN "Manuf. Part"
 	1    5650 1900
 	1    0    0    -1
@@
 F 0 "R12" V 3600 1150 50  0000 L CNN
 F 1 "2.1" V 3500 1125 50  0000 L CNN
-F 2 "" V 3530 1200 50  0001 C CNN
-F 3 "" H 3600 1200 50  0001 C CNN
+F 2 "Resistor_SMD:R_0603_1608Metric_Pad1.05x0.95mm_HandSolder" V 3530 1200 50  0001 C CNN
+F 3 "https://datasheet.lcsc.com/szlcsc/1811082014_YAGEO-RC0603FR-072K1L_C245950.pdf" H 3600 1200 50  0001 C CNN
 F 4 "lcsc.com" H 3600 1200 50  0001 C CNN "Distributor"
-F 5 "RK73B2ATTD102J" H 3600 1200 50  0001 C CNN "Manuf. Part"
+F 5 "RC0603FR-072K1L" H 3600 1200 50  0001 C CNN "Manuf. Part"
 	1    3600 1200
 	0    -1   -1   0
@@
 F 0 "R10" H 5709 1646 50  0000 L CNN
 F 1 "10k" H 5709 1555 50  0000 L CNN
-F 2 "" H 5650 1600 50  0001 C CNN
-F 3 "" H 5650 1600 50  0001 C CNN
+F 2 "Resistor_SMD:R_0603_1608Metric_Pad1.05x0.95mm_HandSolder" H 5650 1600 50  0001 C CNN
+F 3 "https://datasheet.lcsc.com/szlcsc/2004232133_ROHM-Semicon-SFR03EZPF1002_C510290.pdf" H 5650 1600 50  0001 C CNN
 F 4 "lcsc.com" H 5650 1600 50  0001 C CNN "Distributor"
-F 5 "RK73B2ATTD102J" H 5650 1600 50  0001 C CNN "Manuf. Part"
+F 5 "SFR03EZPF1002" H 5650 1600 50  0001 C CNN "Manuf. Part"
 	1    5650 1600
 	1    0    0    -1
@@
 F 0 "R13" V 4000 1150 50  0000 L CNN
 F 1 "0.01" V 4100 1125 50  0000 L CNN
-F 2 "" V 3930 1200 50  0001 C CNN
-F 3 "" H 4000 1200 50  0001 C CNN
+F 2 "Resistor_SMD:R_2512_6332Metric_Pad1.52x3.35mm_HandSolder" V 3930 1200 50  0001 C CNN
+F 3 "https://datasheet.lcsc.com/szlcsc/2008171235_YAGEO-RL2512JK-070R01L_C705618.pdf" H 4000 1200 50  0001 C CNN
 F 4 "lcsc.com" H 4000 1200 50  0001 C CNN "Distributor"
-F 5 "RK73B2ATTD102J" H 4000 1200 50  0001 C CNN "Manuf. Part"
+F 5 "RL2512JK-070R01L" H 4000 1200 50  0001 C CNN "Manuf. Part"
 	1    4000 1200
 	0    1    1    0
@@
 F 0 "R14" H 6059 1446 50  0000 L CNN
 F 1 "10k" H 6059 1355 50  0000 L CNN
-F 2 "" H 6000 1400 50  0001 C CNN
-F 3 "" H 6000 1400 50  0001 C CNN
+F 2 "Resistor_SMD:R_0603_1608Metric_Pad1.05x0.95mm_HandSolder" H 6000 1400 50  0001 C CNN
+F 3 "https://datasheet.lcsc.com/szlcsc/2004232133_ROHM-Semicon-SFR03EZPF1002_C510290.pdf" H 6000 1400 50  0001 C CNN
 F 4 "lcsc.com" H 6000 1400 50  0001 C CNN "Distributor"
-F 5 "RK73B2ATTD102J" H 6000 1400 50  0001 C CNN "Manuf. Part"
+F 5 "SFR03EZPF1002" H 6000 1400 50  0001 C CNN "Manuf. Part"
 	1    6000 1400
 	1    0    0    -1

Commit message: add(hw): more BOM updates
Parts:
- C1: value 10uF -> x
- C10, C8: Manuf. Part TAJA106K016RNJ -> (none)
- C11: value 1uF -> 1nF; footprint (none) -> Capacitor_SMD:C_0603_1608Metric_Pad1.05x0.95mm_HandSolder; Manuf. Part CL21A106MQFNNNE -> CC0402KRX7R0BB102
- C6: value 33uF -> 4.7uF; footprint (none) -> Capacitor_SMD:C_1210_3225Metric_Pad1.42x2.65mm_HandSolder; Manuf. Part TAJA106K016RNJ -> C3225X7S2A475KT000N
- C7: value 1uF -> 680nF; footprint (none) -> Capacitor_SMD:C_0805_2012Metric_Pad1.15x1.40mm_HandSolder; Manuf. Part CL21A106MQFNNNE -> CC0805KKX7R9BB684
- C9: Manuf. Part CL21A106MQFNNNE -> (none)
- D5: value B540C -> MBRB2060; footprint Diode_SMD:D_SMC -> Diode_SMD:D_Powermite3; Manuf. Part B540C-13-F -> MBRB2060CT
Changed lines of the file:
@@
 P 3650 2300
 F 0 "C1" H 3765 2346 50  0000 L CNN
-F 1 "10uF" H 3765 2255 50  0000 L CNN
+F 1 "x" H 3765 2255 50  0000 L CNN
 F 2 "Capacitor_Tantalum_SMD:CP_EIA-3216-18_Kemet-A_Pad1.58x1.35mm_HandSolder" H 3650 2300 50  0001 C CNN
 F 3 "https://datasheet.lcsc.com/szlcsc/AVX-TAJA106K016RNJ_C7171.pdf" H 3650 2300 50  0001 C CNN
@@
 F 1 "330uF" H 1965 5505 50  0000 L CNN
 F 2 "" H 1888 5400 50  0001 C CNN
-F 3 "~" H 1850 5550 50  0001 C CNN
+F 3 "" H 1850 5550 50  0001 C CNN
 	1    1850 5550
 	1    0    0    -1
@@
 F 3 "" H 5250 1450 50  0001 C CNN
 F 4 "lcsc.com" H 5250 1450 50  0001 C CNN "Distributor"
-F 5 "CL21A106MQFNNNE" H 5250 1450 50  0001 C CNN "Manuf. Part"
+F 5 "" H 5250 1450 50  0001 C CNN "Manuf. Part"
 	1    5250 1450
 	1    0    0    -1
@@
 P 4750 1350
 F 0 "D5" V 4704 1430 50  0000 L CNN
-F 1 "B540C" V 4795 1430 50  0000 L CNN
-F 2 "Diode_SMD:D_SMC" H 4750 1350 50  0001 C CNN
-F 3 "https://datasheet.lcsc.com/szlcsc/1810101831_Diodes-Incorporated-B540C-13-F_C72264.pdf" H 4750 1350 50  0001 C CNN
+F 1 "MBRB2060" V 4795 1430 50  0000 L CNN
+F 2 "Diode_SMD:D_Powermite3" H 4750 1350 50  0001 C CNN
+F 3 "https://datasheet.lcsc.com/szlcsc/Sangdest-Microelectronicstronic-Nanjing-MBRB2060CT_C260296.pdf" H 4750 1350 50  0001 C CNN
 F 4 "lcsc.com" H 4750 1350 50  0001 C CNN "Distributor"
-F 5 "B540C-13-F" H 4750 1350 50  0001 C CNN "Manuf. Part"
+F 5 "MBRB2060CT" H 4750 1350 50  0001 C CNN "Manuf. Part"
 	1    4750 1350
 	0    1    1    0
@@
 F 3 "" H 6000 1725 50  0001 C CNN
 F 4 "lcsc.com" H 6000 1725 50  0001 C CNN "Distributor"
-F 5 "TAJA106K016RNJ" H 6000 1725 50  0001 C CNN "Manuf. Part"
+F 5 "" H 6000 1725 50  0001 C CNN "Manuf. Part"
 	1    6000 1725
 	1    0    0    -1
@@
 P 1625 1250
 F 0 "C6" H 1725 1300 50  0000 L CNN
-F 1 "33uF" H 1725 1200 50  0000 L CNN
-F 2 "" H 1625 1250 50  0001 C CNN
-F 3 "" H 1625 1250 50  0001 C CNN
+F 1 "4.7uF" H 1725 1200 50  0000 L CNN
+F 2 "Capacitor_SMD:C_1210_3225Metric_Pad1.42x2.65mm_HandSolder" H 1625 1250 50  0001 C CNN
+F 3 "https://datasheet.lcsc.com/szlcsc/1912111437_TDK-C3225X7S2A475KT000N_C342614.pdf" H 1625 1250 50  0001 C CNN
 F 4 "lcsc.com" H 1625 1250 50  0001 C CNN "Distributor"
-F 5 "TAJA106K016RNJ" H 1625 1250 50  0001 C CNN "Manuf. Part"
+F 5 "C3225X7S2A475KT000N" H 1625 1250 50  0001 C CNN "Manuf. Part"
 	1    1625 1250
 	1    0    0    -1
@@
 P 3600 1050
 F 0 "C11" H 3350 1050 50  0000 L CNN
-F 1 "1uF" H 3350 1150 50  0000 L CNN
-F 2 "" H 3638 900 50  0001 C CNN
-F 3 "" H 3600 1050 50  0001 C CNN
+F 1 "1nF" H 3350 1150 50  0000 L CNN
+F 2 "Capacitor_SMD:C_0603_1608Metric_Pad1.05x0.95mm_HandSolder" H 3638 900 50  0001 C CNN
+F 3 "https://datasheet.lcsc.com/szlcsc/2005222139_YAGEO-CC0402KRX7R0BB102_C527013.pdf" H 3600 1050 50  0001 C CNN
 F 4 "lcsc.com" H 3600 1050 50  0001 C CNN "Distributor"
-F 5 "CL21A106MQFNNNE" H 3600 1050 50  0001 C CNN "Manuf. Part"
+F 5 "CC0402KRX7R0BB102" H 3600 1050 50  0001 C CNN "Manuf. Part"
 	1    3600 1050
 	0    1    1    0
@@
 F 3 "" H 3450 850 50  0001 C CNN
 F 4 "lcsc.com" H 3450 850 50  0001 C CNN "Distributor"
-F 5 "TAJA106K016RNJ" H 3450 850 50  0001 C CNN "Manuf. Part"
+F 5 "" H 3450 850 50  0001 C CNN "Manuf. Part"
 	1    3450 850
 	1    0    0    -1
@@
 P 2200 1250
 F 0 "C7" H 2000 1300 50  0000 L CNN
-F 1 "1uF" H 1950 1200 50  0000 L CNN
-F 2 "" H 2238 1100 50  0001 C CNN
-F 3 "" H 2200 1250 50  0001 C CNN
+F 1 "680nF" H 1950 1200 50  0000 L CNN
+F 2 "Capacitor_SMD:C_0805_2012Metric_Pad1.15x1.40mm_HandSolder" H 2238 1100 50  0001 C CNN
+F 3 "https://datasheet.lcsc.com/szlcsc/1810311413_YAGEO-CC0805KKX7R9BB684_C107133.pdf" H 2200 1250 50  0001 C CNN
 F 4 "lcsc.com" H 2200 1250 50  0001 C CNN "Distributor"
-F 5 "CL21A106MQFNNNE" H 2200 1250 50  0001 C CNN "Manuf. Part"
+F 5 "CC0805KKX7R9BB684" H 2200 1250 50  0001 C CNN "Manuf. Part"
 	1    2200 1250
 	1    0    0    -1

Commit message: add(hw): more footprints and boms
Parts:
- R1, R2, R3, R4, R5, R6, R7: Manuf. Part RK73B2ATTD102J -> RC0805FR-071KL
- R10, R14: Manuf. Part SFR03EZPF1002 -> RC0805FR-0710KL
- R12: value 2.1 -> 2.1k
Changed lines of the file:
@@
 F 1 "1k" H 5159 2255 50  0000 L CNN
 F 2 "Resistor_SMD:R_0805_2012Metric_Pad1.15x1.40mm_HandSolder" H 5100 2300 50  0001 C CNN
-F 3 "https://datasheet.lcsc.com/szlcsc/1810301711_KOA-Speer-Elec-RK73B2ATTD102J_C159911.pdf" H 5100 2300 50  0001 C CNN
+F 3 "https://datasheet.lcsc.com/szlcsc/1810010118_YAGEO-RC0805FR-071KL_C95781.pdf" H 5100 2300 50  0001 C CNN
 F 4 "lcsc.com" H 5100 2300 50  0001 C CNN "Distributor"
-F 5 "RK73B2ATTD102J" H 5100 2300 50  0001 C CNN "Manuf. Part"
+F 5 " 	RC0805FR-071KL" H 5100 2300 50  0001 C CNN "Manuf. Part"
 	1    5100 2300
 	1    0    0    -1
@@
 F 1 "1k" H 7859 5005 50  0000 L CNN
 F 2 "Resistor_SMD:R_0805_2012Metric_Pad1.15x1.40mm_HandSolder" H 7800 5050 50  0001 C CNN
-F 3 "https://datasheet.lcsc.com/szlcsc/1810301711_KOA-Speer-Elec-RK73B2ATTD102J_C159911.pdf" H 7800 5050 50  0001 C CNN
+F 3 "https://datasheet.lcsc.com/szlcsc/1810010118_YAGEO-RC0805FR-071KL_C95781.pdf" H 7800 5050 50  0001 C CNN
 F 4 "lcsc.com" H 7800 5050 50  0001 C CNN "Distributor"
-F 5 "RK73B2ATTD102J" H 7800 5050 50  0001 C CNN "Manuf. Part"
+F 5 " 	RC0805FR-071KL" H 7800 5050 50  0001 C CNN "Manuf. Part"
 	1    7800 5050
 	1    0    0    -1
@@
 F 1 "1k" H 1700 3950 50  0000 L CNN
 F 2 "Resistor_SMD:R_0805_2012Metric_Pad1.15x1.40mm_HandSolder" H 1850 4000 50  0001 C CNN
-F 3 "https://datasheet.lcsc.com/szlcsc/1810301711_KOA-Speer-Elec-RK73B2ATTD102J_C159911.pdf" H 1850 4000 50  0001 C CNN
+F 3 "https://datasheet.lcsc.com/szlcsc/1810010118_YAGEO-RC0805FR-071KL_C95781.pdf" H 1850 4000 50  0001 C CNN
 F 4 "lcsc.com" H 1850 4000 50  0001 C CNN "Distributor"
-F 5 "RK73B2ATTD102J" H 1850 4000 50  0001 C CNN "Manuf. Part"
+F 5 " 	RC0805FR-071KL" H 1850 4000 50  0001 C CNN "Manuf. Part"
 	1    1850 4000
 	1    0    0    -1
@@
 F 1 "1k" H 2100 3950 50  0000 L CNN
 F 2 "Resistor_SMD:R_0805_2012Metric_Pad1.15x1.40mm_HandSolder" H 2050 4000 50  0001 C CNN
-F 3 "https://datasheet.lcsc.com/szlcsc/1810301711_KOA-Speer-Elec-RK73B2ATTD102J_C159911.pdf" H 2050 4000 50  0001 C CNN
+F 3 "https://datasheet.lcsc.com/szlcsc/1810010118_YAGEO-RC0805FR-071KL_C95781.pdf" H 2050 4000 50  0001 C CNN
 F 4 "lcsc.com" H 2050 4000 50  0001 C CNN "Distributor"
-F 5 "RK73B2ATTD102J" H 2050 4000 50  0001 C CNN "Manuf. Part"
+F 5 " 	RC0805FR-071KL" H 2050 4000 50  0001 C CNN "Manuf. Part"
 	1    2050 4000
 	1    0    0    -1
@@
 F 1 "1k" H 7759 5005 50  0000 L CNN
 F 2 "Resistor_SMD:R_0805_2012Metric_Pad1.15x1.40mm_HandSolder" H 7700 5050 50  0001 C CNN
-F 3 "https://datasheet.lcsc.com/szlcsc/1810301711_KOA-Speer-Elec-RK73B2ATTD102J_C159911.pdf" H 7700 5050 50  0001 C CNN
+F 3 "https://datasheet.lcsc.com/szlcsc/1810010118_YAGEO-RC0805FR-071KL_C95781.pdf" H 7700 5050 50  0001 C CNN
 F 4 "lcsc.com" H 7700 5050 50  0001 C CNN "Distributor"
-F 5 "RK73B2ATTD102J" H 7700 5050 50  0001 C CNN "Manuf. Part"
+F 5 " 	RC0805FR-071KL" H 7700 5050 50  0001 C CNN "Manuf. Part"
 	1    7700 5050
 	-1   0    0    1
@@
 F 1 "1k" H 9159 2705 50  0000 L CNN
 F 2 "Resistor_SMD:R_0805_2012Metric_Pad1.15x1.40mm_HandSolder" H 9100 2750 50  0001 C CNN
-F 3 "https://datasheet.lcsc.com/szlcsc/1810301711_KOA-Speer-Elec-RK73B2ATTD102J_C159911.pdf" H 9100 2750 50  0001 C CNN
+F 3 "https://datasheet.lcsc.com/szlcsc/1810010118_YAGEO-RC0805FR-071KL_C95781.pdf" H 9100 2750 50  0001 C CNN
 F 4 "lcsc.com" H 9100 2750 50  0001 C CNN "Distributor"
-F 5 "RK73B2ATTD102J" H 9100 2750 50  0001 C CNN "Manuf. Part"
+F 5 " 	RC0805FR-071KL" H 9100 2750 50  0001 C CNN "Manuf. Part"
 	1    9100 2750
 	1    0    0    -1
@@
 F 1 "1k" H 1459 4755 50  0000 L CNN
 F 2 "Resistor_SMD:R_0805_2012Metric_Pad1.15x1.40mm_HandSolder" H 1400 4800 50  0001 C CNN
-F 3 "https://datasheet.lcsc.com/szlcsc/1810301711_KOA-Speer-Elec-RK73B2ATTD102J_C159911.pdf" H 1400 4800 50  0001 C CNN
+F 3 "https://datasheet.lcsc.com/szlcsc/1810010118_YAGEO-RC0805FR-071KL_C95781.pdf" H 1400 4800 50  0001 C CNN
 F 4 "lcsc.com" H 1400 4800 50  0001 C CNN "Distributor"
-F 5 "RK73B2ATTD102J" H 1400 4800 50  0001 C CNN "Manuf. Part"
+F 5 " 	RC0805FR-071KL" H 1400 4800 50  0001 C CNN "Manuf. Part"
 	1    1400 4800
 	1    0    0    -1
@@
 P 1625 1250
 F 0 "C6" H 1725 1300 50  0000 L CNN
-F 1 "4.7uF" H 1725 1200 50  0000 L CNN
+F 1 "4.7uF" H 1675 1150 50  0000 L CNN
 F 2 "Capacitor_SMD:C_1210_3225Metric_Pad1.42x2.65mm_HandSolder" H 1625 1250 50  0001 C CNN
 F 3 "https://datasheet.lcsc.com/szlcsc/1912111437_TDK-C3225X7S2A475KT000N_C342614.pdf" H 1625 1250 50  0001 C CNN
@@
 U 1 1 5FEEDDCD
 P 3600 1200
-F 0 "R12" V 3600 1150 50  0000 L CNN
-F 1 "2.1" V 3500 1125 50  0000 L CNN
+F 0 "R12" V 3600 1125 50  0000 L CNN
+F 1 "2.1k" V 3500 1125 50  0000 L CNN
 F 2 "Resistor_SMD:R_0603_1608Metric_Pad1.05x0.95mm_HandSolder" V 3530 1200 50  0001 C CNN
 F 3 "https://datasheet.lcsc.com/szlcsc/1811082014_YAGEO-RC0603FR-072K1L_C245950.pdf" H 3600 1200 50  0001 C CNN
@@
 F 1 "10k" H 5709 1555 50  0000 L CNN
 F 2 "Resistor_SMD:R_0603_1608Metric_Pad1.05x0.95mm_HandSolder" H 5650 1600 50  0001 C CNN
-F 3 "https://datasheet.lcsc.com/szlcsc/2004232133_ROHM-Semicon-SFR03EZPF1002_C510290.pdf" H 5650 1600 50  0001 C CNN
+F 3 "https://datasheet.lcsc.com/szlcsc/1810201611_YAGEO-RC0805FR-0710KL_C84376.pdf" H 5650 1600 50  0001 C CNN
 F 4 "lcsc.com" H 5650 1600 50  0001 C CNN "Distributor"
-F 5 "SFR03EZPF1002" H 5650 1600 50  0001 C CNN "Manuf. Part"
+F 5 "RC0805FR-0710KL" H 5650 1600 50  0001 C CNN "Manuf. Part"
 	1    5650 1600
 	1    0    0    -1
@@
 P 2200 1250
 F 0 "C7" H 2000 1300 50  0000 L CNN
-F 1 "680nF" H 1950 1200 50  0000 L CNN
+F 1 "680nF" H 1950 1150 50  0000 L CNN
 F 2 "Capacitor_SMD:C_0805_2012Metric_Pad1.15x1.40mm_HandSolder" H 2238 1100 50  0001 C CNN
 F 3 "https://datasheet.lcsc.com/szlcsc/1810311413_YAGEO-CC0805KKX7R9BB684_C107133.pdf" H 2200 1250 50  0001 C CNN
@@
 U 1 1 5FEAD2F6
 P 4000 1200
-F 0 "R13" V 4000 1150 50  0000 L CNN
+F 0 "R13" V 3900 1125 50  0000 L CNN
 F 1 "0.01" V 4100 1125 50  0000 L CNN
 F 2 "Resistor_SMD:R_2512_6332Metric_Pad1.52x3.35mm_HandSolder" V 3930 1200 50  0001 C CNN
@@
 F 1 "10k" H 6059 1355 50  0000 L CNN
 F 2 "Resistor_SMD:R_0603_1608Metric_Pad1.05x0.95mm_HandSolder" H 6000 1400 50  0001 C CNN
-F 3 "https://datasheet.lcsc.com/szlcsc/2004232133_ROHM-Semicon-SFR03EZPF1002_C510290.pdf" H 6000 1400 50  0001 C CNN
+F 3 "https://datasheet.lcsc.com/szlcsc/1810201611_YAGEO-RC0805FR-0710KL_C84376.pdf" H 6000 1400 50  0001 C CNN
 F 4 "lcsc.com" H 6000 1400 50  0001 C CNN "Distributor"
-F 5 "SFR03EZPF1002" H 6000 1400 50  0001 C CNN "Manuf. Part"
+F 5 "RC0805FR-0710KL" H 6000 1400 50  0001 C CNN "Manuf. Part"
 	1    6000 1400
 	1    0    0    -1
