File: hw/blueled.sch (KiCad schematic (older format))
At the start: 58 parts, among them J1 Barrel_Jack, J2 LED Strip, J3 ICSP, J4 Screw_Terminal_01x02, Q1 Q_PMOS_SDG, Q2 Q_PNP_EBC, SW2 PUSH, U1 ATmega328P-AU, U2 HC-05, U3 AMS1117-3.3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

Commit message: add(hw): minor adjacements of output filter
Parts:
- added C13: 47uF, Capacitor_SMD:C_1210_3225Metric_Pad1.42x2.65mm_HandSolder, symbol Device:CP1
- C10: value 100uF -> 47uF; footprint Capacitor_SMD:C_1206_3216Metric_Pad1.42x1.75mm_HandSolder -> Capacitor_SMD:C_1210_3225Metric_Pad1.42x2.65mm_HandSolder; Manuf. Part GRM31CR60J107ME39L -> C3225X5R0J476MT000N
- C6: footprint Capacitor_SMD:C_1206_3216Metric_Pad1.42x1.75mm_HandSolder -> Capacitor_SMD:C_1210_3225Metric_Pad1.42x2.65mm_HandSolder; Manuf. Part CGA5L3X7S2A225KT0Y0N -> C3225X7S2A475KT000N
- C9: value 0.1uF -> 4700pF
- R14: value 10k -> 0.27; Manuf. Part RC0805FR-0710KL -> RL0805JR-070R27L
Connections:
- net GND: now also C13.2
- net at C10.1, R14.2: now also C13.1
Other:
- moved on the sheet: D4, R15
Changed lines of the file:
@@
 U 1 1 5FE1A9BA
 P 5250 1450
-F 0 "C9" H 5400 1500 50  0000 L CNN
-F 1 "0.1uF" H 5400 1400 50  0000 L CNN
+F 0 "C9" H 5350 1500 50  0000 L CNN
+F 1 "4700pF" H 5325 1400 50  0000 L CNN
 F 2 "Capacitor_SMD:C_0805_2012Metric_Pad1.15x1.40mm_HandSolder" H 5288 1300 50  0001 C CNN
 F 3 "https://datasheet.lcsc.com/szlcsc/1912111437_TDK-C2012C0G1H472JT0H0N_C342964.pdf" H 5250 1450 50  0001 C CNN
@@
 U 1 1 5FE3F026
 P 4750 1350
-F 0 "D5" V 4704 1430 50  0000 L CNN
-F 1 "MBRB2060" V 4795 1430 50  0000 L CNN
+F 0 "D5" V 4700 1425 50  0000 L CNN
+F 1 "MBRB2060" V 4775 1425 50  0000 L CNN
 F 2 "Diode_SMD:D_Powermite3" H 4750 1350 50  0001 C CNN
 F 3 "https://datasheet.lcsc.com/szlcsc/Sangdest-Microelectronicstronic-Nanjing-MBRB2060CT_C260296.pdf" H 4750 1350 50  0001 C CNN
@@
 U 1 1 5FE853F6
 P 6000 1725
-F 0 "C10" H 6115 1771 50  0000 L CNN
-F 1 "100uF" H 6115 1680 50  0000 L CNN
-F 2 "Capacitor_SMD:C_1206_3216Metric_Pad1.42x1.75mm_HandSolder" H 6000 1725 50  0001 C CNN
-F 3 "https://datasheet.lcsc.com/szlcsc/1810201321_Murata-Electronics-GRM31CR60J107ME39L_C77085.pdf" H 6000 1725 50  0001 C CNN
+F 0 "C10" H 6025 1825 50  0000 L CNN
+F 1 "47uF" H 6025 1600 50  0000 L CNN
+F 2 "Capacitor_SMD:C_1210_3225Metric_Pad1.42x2.65mm_HandSolder" H 6000 1725 50  0001 C CNN
+F 3 "https://datasheet.lcsc.com/szlcsc/1912111437_TDK-C3225X5R0J476MT000N_C338024.pdf" H 6000 1725 50  0001 C CNN
 F 4 "lcsc.com" H 6000 1725 50  0001 C CNN "Distributor"
-F 5 "GRM31CR60J107ME39L" H 6000 1725 50  0001 C CNN "Manuf. Part"
+F 5 "C3225X5R0J476MT000N" H 6000 1725 50  0001 C CNN "Manuf. Part"
 	1    6000 1725
 	1    0    0    -1
@@
 L power:+5V #PWR020
 U 1 1 5FF5B0B2
-P 6450 1100
-F 0 "#PWR020" H 6450 950 50  0001 C CNN
-F 1 "+5V" H 6465 1273 50  0000 C CNN
-F 2 "" H 6450 1100 50  0001 C CNN
-F 3 "" H 6450 1100 50  0001 C CNN
-	1    6450 1100
+P 6575 1075
+F 0 "#PWR020" H 6575 925 50  0001 C CNN
+F 1 "+5V" H 6590 1248 50  0000 C CNN
+F 2 "" H 6575 1075 50  0001 C CNN
+F 3 "" H 6575 1075 50  0001 C CNN
+	1    6575 1075
 	1    0    0    -1
 $EndComp
@@
 F 0 "C6" H 1725 1300 50  0000 L CNN
 F 1 "4.7uF" H 1675 1150 50  0000 L CNN
-F 2 "Capacitor_SMD:C_1206_3216Metric_Pad1.42x1.75mm_HandSolder" H 1625 1250 50  0001 C CNN
-F 3 "https://datasheet.lcsc.com/szlcsc/1912111437_TDK-CGA5L3X7S2A225KT0Y0N_C342669.pdf" H 1625 1250 50  0001 C CNN
+F 2 "Capacitor_SMD:C_1210_3225Metric_Pad1.42x2.65mm_HandSolder" H 1625 1250 50  0001 C CNN
+F 3 "https://datasheet.lcsc.com/szlcsc/1903111833_TDK-C3225X7S2A475KT000N_C342614.pdf" H 1625 1250 50  0001 C CNN
 F 4 "lcsc.com" H 1625 1250 50  0001 C CNN "Distributor"
-F 5 "CGA5L3X7S2A225KT0Y0N" H 1625 1250 50  0001 C CNN "Manuf. Part"
+F 5 "C3225X7S2A475KT000N" H 1625 1250 50  0001 C CNN "Manuf. Part"
 	1    1625 1250
 	1    0    0    -1
@@
 Connection ~ 3450 1200
 Wire Wire Line
-	6000 1975 6000 1875
+	6000 1975 6000 1900
 Wire Wire Line
 	4650 1200 4750 1200
@@
 	0    -1   -1   0
 $EndComp
-Wire Wire Line
-	6450 1100 6450 1200
 Wire Wire Line
 	6000 1200 6000 1300
@@
 P 6000 1400
 F 0 "R14" H 6059 1446 50  0000 L CNN
-F 1 "10k" H 6059 1355 50  0000 L CNN
+F 1 "0.27" H 6059 1355 50  0000 L CNN
 F 2 "Resistor_SMD:R_0805_2012Metric_Pad1.15x1.40mm_HandSolder" H 6000 1400 50  0001 C CNN
-F 3 "https://datasheet.lcsc.com/szlcsc/1810201611_YAGEO-RC0805FR-0710KL_C84376.pdf" H 6000 1400 50  0001 C CNN
+F 3 "https://datasheet.lcsc.com/szlcsc/2009282237_YAGEO-RL0805JR-070R27L_C705550.pdf" H 6000 1400 50  0001 C CNN
 F 4 "lcsc.com" H 6000 1400 50  0001 C CNN "Distributor"
-F 5 "RC0805FR-0710KL" H 6000 1400 50  0001 C CNN "Manuf. Part"
+F 5 "RL0805JR-070R27L" H 6000 1400 50  0001 C CNN "Manuf. Part"
 	1    6000 1400
 	1    0    0    -1
 $EndComp
 Wire Wire Line
-	6000 1575 6000 1500
+	6000 1575 6000 1550
 Text Notes 2825 2775 0    50   ~ 0
 Switch off \npower
@@
 L Device:R_Small R15
 U 1 1 5FF22C54
-P 6450 1400
-F 0 "R15" H 6509 1446 50  0000 L CNN
-F 1 "470" H 6509 1355 50  0000 L CNN
-F 2 "Resistor_SMD:R_0805_2012Metric_Pad1.15x1.40mm_HandSolder" H 6450 1400 50  0001 C CNN
-F 3 "https://datasheet.lcsc.com/szlcsc/1810311431_YAGEO-RC0805FR-07470RL_C114564.pdf" H 6450 1400 50  0001 C CNN
-F 4 "lcsc.com" H 6450 1400 50  0001 C CNN "Distributor"
-F 5 "RC0805FR-07470RL" H 6450 1400 50  0001 C CNN "Manuf. Part"
-	1    6450 1400
+P 6575 1400
+F 0 "R15" H 6634 1446 50  0000 L CNN
+F 1 "470" H 6634 1355 50  0000 L CNN
+F 2 "Resistor_SMD:R_0805_2012Metric_Pad1.15x1.40mm_HandSolder" H 6575 1400 50  0001 C CNN
+F 3 "https://datasheet.lcsc.com/szlcsc/1810311431_YAGEO-RC0805FR-07470RL_C114564.pdf" H 6575 1400 50  0001 C CNN
+F 4 "lcsc.com" H 6575 1400 50  0001 C CNN "Distributor"
+F 5 "RC0805FR-07470RL" H 6575 1400 50  0001 C CNN "Manuf. Part"
+	1    6575 1400
 	1    0    0    -1
 $EndComp
@@
 L Device:LED D4
 U 1 1 5FF22C5C
-P 6450 1700
-F 0 "D4" V 6489 1583 50  0000 R CNN
-F 1 "+5V" V 6398 1583 50  0000 R CNN
-F 2 "LED_SMD:LED_0805_2012Metric_Pad1.15x1.40mm_HandSolder" H 6450 1700 50  0001 C CNN
-F 3 "https://datasheet.lcsc.com/szlcsc/1811141223_TOGIALED-TJ-S1608SW6TGLC2G-A5_C192316.pdf" H 6450 1700 50  0001 C CNN
-F 4 "lcsc.com" H 6450 1700 50  0001 C CNN "Distributor"
-F 5 "TJ-S1608SW6TGLC2G-A5 " H 6450 1700 50  0001 C CNN "Manuf. Part"
-	1    6450 1700
-	0    -1   -1   0
-$EndComp
-Wire Wire Line
-	6450 1500 6450 1550
+P 6575 1700
+F 0 "D4" V 6614 1583 50  0000 R CNN
+F 1 "+5V" V 6523 1583 50  0000 R CNN
+F 2 "LED_SMD:LED_0805_2012Metric_Pad1.15x1.40mm_HandSolder" H 6575 1700 50  0001 C CNN
+F 3 "https://datasheet.lcsc.com/szlcsc/1811141223_TOGIALED-TJ-S1608SW6TGLC2G-A5_C192316.pdf" H 6575 1700 50  0001 C CNN
+F 4 "lcsc.com" H 6575 1700 50  0001 C CNN "Distributor"
+F 5 "TJ-S1608SW6TGLC2G-A5 " H 6575 1700 50  0001 C CNN "Manuf. Part"
+	1    6575 1700
+	0    -1   -1   0
+$EndComp
+Wire Wire Line
+	6575 1500 6575 1550
 $Comp
 L power:GND #PWR024
 U 1 1 5FF22C63
-P 6450 1975
-F 0 "#PWR024" H 6450 1725 50  0001 C CNN
-F 1 "GND" H 6455 1802 50  0000 C CNN
-F 2 "" H 6450 1975 50  0001 C CNN
-F 3 "" H 6450 1975 50  0001 C CNN
-	1    6450 1975
-	1    0    0    -1
-$EndComp
-Wire Wire Line
-	6000 1200 6450 1200
-Connection ~ 6000 1200
-Wire Wire Line
-	6450 1300 6450 1200
-Connection ~ 6450 1200
-Wire Wire Line
-	6450 1850 6450 1975
+P 6575 1975
+F 0 "#PWR024" H 6575 1725 50  0001 C CNN
+F 1 "GND" H 6580 1802 50  0000 C CNN
+F 2 "" H 6575 1975 50  0001 C CNN
+F 3 "" H 6575 1975 50  0001 C CNN
+	1    6575 1975
+	1    0    0    -1
+$EndComp
+Wire Wire Line
+	6575 1300 6575 1200
+Wire Wire Line
+	6575 1850 6575 1975
 Wire Wire Line
 	3650 2550 4200 2550
@@
 	5650 1500 5650 1750
 $Comp
-L power:+5V #PWR?
+L power:+5V #PWR0111
 U 1 1 5FEDEB2A
 P 6200 3700
-F 0 "#PWR?" H 6200 3550 50  0001 C CNN
+F 0 "#PWR0111" H 6200 3550 50  0001 C CNN
 F 1 "+5V" H 6215 3873 50  0000 C CNN
 F 2 "" H 6200 3700 50  0001 C CNN
@@
 	1    0    0    -1
 $EndComp
+$Comp
+L Device:CP1 C13
+U 1 1 5FEE1E45
+P 6275 1725
+F 0 "C13" H 6300 1825 50  0000 L CNN
+F 1 "47uF" H 6300 1600 50  0000 L CNN
+F 2 "Capacitor_SMD:C_1210_3225Metric_Pad1.42x2.65mm_HandSolder" H 6275 1725 50  0001 C CNN
+F 3 "https://datasheet.lcsc.com/szlcsc/1912111437_TDK-C3225X5R0J476MT000N_C338024.pdf" H 6275 1725 50  0001 C CNN
+F 4 "lcsc.com" H 6275 1725 50  0001 C CNN "Distributor"
+F 5 "C3225X5R0J476MT000N" H 6275 1725 50  0001 C CNN "Manuf. Part"
+	1    6275 1725
+	1    0    0    -1
+$EndComp
+Wire Wire Line
+	6000 1550 6275 1550
+Wire Wire Line
+	6275 1550 6275 1575
+Connection ~ 6000 1550
+Wire Wire Line
+	6000 1550 6000 1500
+Wire Wire Line
+	6275 1875 6275 1900
+Wire Wire Line
+	6275 1900 6000 1900
+Connection ~ 6000 1900
+Wire Wire Line
+	6000 1900 6000 1875
+Wire Wire Line
+	6000 1200 6575 1200
+Connection ~ 6000 1200
+Wire Wire Line
+	6575 1200 6575 1075
+Connection ~ 6575 1200
 $EndSCHEMATC

Commit message: add(hw): a lot of progress in layouting + bug fixes
Parts:
- D5: footprint Diode_SMD:D_Powermite3 -> Package_TO_SOT_SMD:TO-263-3_TabPin2
Connections:
- net VIN is gone; now on net +5V: C12.1
- net at D5.1 (K), L1.1: now also Q1.2 (D); no longer Q1.1 (S)
- net at R13.1, U5.5 (ISEN): now also Q1.1 (S); no longer Q1.2 (D)
Changed lines of the file:
@@
 F 0 "D5" V 4700 1425 50  0000 L CNN
 F 1 "MBRB2060" V 4775 1425 50  0000 L CNN
-F 2 "Diode_SMD:D_Powermite3" H 4750 1350 50  0001 C CNN
+F 2 "Package_TO_SOT_SMD:TO-263-3_TabPin2" H 4750 1350 50  0001 C CNN
 F 3 "https://datasheet.lcsc.com/szlcsc/Sangdest-Microelectronicstronic-Nanjing-MBRB2060CT_C260296.pdf" H 4750 1350 50  0001 C CNN
 F 4 "lcsc.com" H 4750 1350 50  0001 C CNN "Distributor"
@@
 U 1 1 6068EAC3
 P 5800 4250
-F 0 "C12" V 6050 4250 50  0000 L CNN
-F 1 "1000uF" V 5950 4150 50  0000 L CNN
+F 0 "C12" V 6030 4160 50  0000 L CNN
+F 1 "1000uF" V 5950 4025 50  0000 L CNN
 F 2 "Capacitor_SMD:CP_Elec_10x10" H 5800 4250 50  0001 C CNN
 F 3 "https://datasheet.lcsc.com/szlcsc/1912111437_Lelon-VEU102M0JTR-1010_C249735.pdf" H 5800 4250 50  0001 C CNN
@@
 	0    -1   -1   0
 $EndComp
-Text Label 5550 4250 2    50   ~ 0
-VIN
 Wire Wire Line
 	5550 4250 5650 4250
@@
 Wire Wire Line
 	6000 1975 6000 1900
-Wire Wire Line
-	4650 1200 4750 1200
 Connection ~ 4750 1200
 Wire Wire Line
@@
 Wire Wire Line
 	2200 1400 2200 1500
-$Comp
-L Device:Q_PMOS_SDG Q1
-U 1 1 5D461D8C
-P 4450 1300
-F 0 "Q1" V 4700 1250 50  0000 L CNN
-F 1 "Q_PMOS_SDG" V 4700 1050 50  0001 L CNN
-F 2 "Package_TO_SOT_SMD:TO-252-3_TabPin4" H 4650 1400 50  0001 C CNN
-F 3 "https://datasheet.lcsc.com/szlcsc/Alpha-Omega-Semicon-AOS-AOD4185_C77993.pdf" H 4450 1300 50  0001 C CNN
-F 4 "lcsc.com" H 4450 1300 50  0001 C CNN "Distributor"
-F 5 "AOD4185L" H 4450 1300 50  0001 C CNN "Manuf. Part"
-	1    4450 1300
-	0    -1   -1   0
-$EndComp
 Wire Wire Line
 	6000 1200 6000 1300
@@
 	6575 1200 6575 1075
 Connection ~ 6575 1200
+$Comp
+L power:+5V #PWR0112
+U 1 1 6006B235
+P 5550 4250
+F 0 "#PWR0112" H 5550 4100 50  0001 C CNN
+F 1 "+5V" H 5565 4423 50  0000 C CNN
+F 2 "" H 5550 4250 50  0001 C CNN
+F 3 "" H 5550 4250 50  0001 C CNN
+	1    5550 4250
+	1    0    0    -1
+$EndComp
+Wire Wire Line
+	4650 1200 4750 1200
+$Comp
+L Device:Q_PMOS_SDG Q1
+U 1 1 5D461D8C
+P 4450 1300
+F 0 "Q1" V 4700 1250 50  0000 L CNN
+F 1 "Q_PMOS_SDG" V 4700 1050 50  0001 L CNN
+F 2 "Package_TO_SOT_SMD:TO-252-3_TabPin4" H 4650 1400 50  0001 C CNN
+F 3 "https://datasheet.lcsc.com/szlcsc/Alpha-Omega-Semicon-AOS-AOD4185_C77993.pdf" H 4450 1300 50  0001 C CNN
+F 4 "lcsc.com" H 4450 1300 50  0001 C CNN "Distributor"
+F 5 "AOD4185L" H 4450 1300 50  0001 C CNN "Manuf. Part"
+	1    4450 1300
+	0    1    -1   0
+$EndComp
 $EndSCHEMATC

Commit message: add(hw): level shifter + layout progress
Parts:
- added Q3: BSS138, Package_TO_SOT_SMD:SOT-23, symbol Transistor_FET:BSS138
- added R16, R17: 1k, Resistor_SMD:R_0805_2012Metric_Pad1.15x1.40mm_HandSolder, symbol Device:R_Small
Connections:
- net +3V3: now also Q3.1 (G), R16.1
- net +5V: now also R17.1
- net DATA: now also Q3.3 (D), R17.2; no longer R11.2
- new net: Q3.2 (S), R11.2, R16.2
Other:
- note added: "Level shifter as\nMCU is 3.3V but\nWS2812B needs 5V"
Changed lines of the file:
@@
 Text Label 8950 3650 0    50   ~ 0
 HC-DISCNCT
-Text Label 9250 3850 0    50   ~ 0
+Text Label 10310 3850 0    50   ~ 0
 DATA
 Wire Wire Line
@@
 $EndComp
 Wire Wire Line
-	9750 3050 9750 2950
+	9840 3050 9840 2950
 $Comp
 L blueled-rescue:PUSH-_electromech SW2
@@
 L power:GND #PWR0105
 U 1 1 5CBEBE63
-P 9750 3050
-F 0 "#PWR0105" H 9750 2800 50  0001 C CNN
-F 1 "GND" H 9755 2877 50  0000 C CNN
-F 2 "" H 9750 3050 50  0001 C CNN
-F 3 "" H 9750 3050 50  0001 C CNN
-	1    9750 3050
+P 9840 3050
+F 0 "#PWR0105" H 9840 2800 50  0001 C CNN
+F 1 "GND" H 9845 2877 50  0000 C CNN
+F 2 "" H 9840 3050 50  0001 C CNN
+F 3 "" H 9840 3050 50  0001 C CNN
+	1    9840 3050
 	1    0    0    -1
 $EndComp
@@
 	6950 600  6950 6300
 Wire Notes Line width 12
-	9900 600  9900 6300
+	11080 600  11080 6300
 Wire Notes Line width 12
 	5300 6300 9900 6300
@@
 	0    -1   -1   0
 $EndComp
-Wire Wire Line
-	9150 3850 9250 3850
 $Comp
 L Device:CP1 C12
@@
 	0    1    -1   0
 $EndComp
+$Comp
+L Transistor_FET:BSS138 Q3
+U 1 1 5FF0D3AD
+P 9890 3750
+F 0 "Q3" V 10139 3750 50  0000 C CNN
+F 1 "BSS138" V 10230 3750 50  0000 C CNN
+F 2 "Package_TO_SOT_SMD:SOT-23" H 10090 3675 50  0001 L CIN
+F 3 "https://www.fairchildsemi.com/datasheets/BS/BSS138.pdf" H 9890 3750 50  0001 L CNN
+F 4 "lcsc.com" H 9890 3750 50  0001 C CNN "Distributor"
+F 5 "BSS138" H 9890 3750 50  0001 C CNN "Manuf. Part"
+	1    9890 3750
+	0    1    1    0
+$EndComp
+$Comp
+L Device:R_Small R16
+U 1 1 5FF1EEFC
+P 9600 3650
+F 0 "R16" H 9659 3696 50  0000 L CNN
+F 1 "1k" H 9659 3605 50  0000 L CNN
+F 2 "Resistor_SMD:R_0805_2012Metric_Pad1.15x1.40mm_HandSolder" H 9600 3650 50  0001 C CNN
+F 3 "https://datasheet.lcsc.com/szlcsc/1810010118_YAGEO-RC0805FR-071KL_C95781.pdf" H 9600 3650 50  0001 C CNN
+F 4 "lcsc.com" H 9600 3650 50  0001 C CNN "Distributor"
+F 5 "RC0805FR-071KL" H 9600 3650 50  0001 C CNN "Manuf. Part"
+	1    9600 3650
+	1    0    0    -1
+$EndComp
+$Comp
+L Device:R_Small R17
+U 1 1 5FF2B507
+P 10190 3650
+F 0 "R17" H 10249 3696 50  0000 L CNN
+F 1 "1k" H 10249 3605 50  0000 L CNN
+F 2 "Resistor_SMD:R_0805_2012Metric_Pad1.15x1.40mm_HandSolder" H 10190 3650 50  0001 C CNN
+F 3 "https://datasheet.lcsc.com/szlcsc/1810010118_YAGEO-RC0805FR-071KL_C95781.pdf" H 10190 3650 50  0001 C CNN
+F 4 "lcsc.com" H 10190 3650 50  0001 C CNN "Distributor"
+F 5 "RC0805FR-071KL" H 10190 3650 50  0001 C CNN "Manuf. Part"
+	1    10190 3650
+	1    0    0    -1
+$EndComp
+$Comp
+L power:+5V #PWR026
+U 1 1 5FFE7891
+P 10190 3400
+F 0 "#PWR026" H 10190 3250 50  0001 C CNN
+F 1 "+5V" H 10205 3573 50  0000 C CNN
+F 2 "" H 10190 3400 50  0001 C CNN
+F 3 "" H 10190 3400 50  0001 C CNN
+	1    10190 3400
+	1    0    0    -1
+$EndComp
+Wire Wire Line
+	9750 2950 9840 2950
+Wire Wire Line
+	9150 3850 9600 3850
+$Comp
+L power:+3.3V #PWR025
+U 1 1 60161DE9
+P 9600 3400
+F 0 "#PWR025" H 9600 3250 50  0001 C CNN
+F 1 "+3.3V" H 9615 3573 50  0000 C CNN
+F 2 "" H 9600 3400 50  0001 C CNN
+F 3 "" H 9600 3400 50  0001 C CNN
+	1    9600 3400
+	1    0    0    -1
+$EndComp
+Wire Wire Line
+	9600 3750 9600 3850
+Connection ~ 9600 3850
+Wire Wire Line
+	9600 3850 9690 3850
+Wire Wire Line
+	9600 3400 9600 3470
+Wire Wire Line
+	9600 3470 9890 3470
+Wire Wire Line
+	9890 3470 9890 3550
+Connection ~ 9600 3470
+Wire Wire Line
+	9600 3470 9600 3550
+Wire Notes Line width 12
+	9910 600  11090 600
+Wire Notes Line width 12
+	9910 4550 11090 4550
+Wire Notes Line width 12
+	9910 6300 11090 6300
+Wire Notes Line
+	11080 6300 11080 6290
+Text Notes 10170 4210 0    50   ~ 0
+Level shifter as\nMCU is 3.3V but\nWS2812B needs 5V
+Wire Wire Line
+	10090 3850 10190 3850
+Wire Wire Line
+	10190 3750 10190 3850
+Connection ~ 10190 3850
+Wire Wire Line
+	10190 3850 10310 3850
+Wire Wire Line
+	10190 3400 10190 3550
 $EndSCHEMATC

Commit message: fix(hw): change input cap + minor fixes
Parts:
- C6: value 4.7uF -> 33uF; footprint Capacitor_SMD:C_1210_3225Metric_Pad1.42x2.65mm_HandSolder -> Capacitor_SMD:CP_Elec_10x10; Manuf. Part C3225X7S2A475KT000N -> VZH330M2ATR-1010

Commit message: fix(hw): minor adjustments (shorter current loop)
Parts:
- D2: value LED -> RX
- D3: value LED -> TX
- J1: value Barrel_Jack -> DC 5.5 - 42V
- J4: value Screw_Terminal_01x02 -> DC 5.5 - 42V
Changed lines of the file:
@@
 P 950 1100
 F 0 "J1" H 1007 1425 50  0000 C CNN
-F 1 "Barrel_Jack" H 1007 1334 50  0000 C CNN
+F 1 "DC 5.5 - 42V" H 1007 1334 50  0000 C CNN
 F 2 "Connector_BarrelJack:BarrelJack_Horizontal" H 1000 1060 50  0001 C CNN
 F 3 "https://datasheet.lcsc.com/szlcsc/1912111437_XKB-Enterprise-DC-005-5A-2-0_C381116.pdf" H 1000 1060 50  0001 C CNN
@@
 P 1850 3700
 F 0 "D3" V 1900 3900 50  0000 R CNN
-F 1 "LED" V 1800 3900 50  0000 R CNN
+F 1 "TX" V 1800 3900 50  0000 R CNN
 F 2 "LED_SMD:LED_0805_2012Metric_Pad1.15x1.40mm_HandSolder" H 1850 3700 50  0001 C CNN
 F 3 "https://datasheet.lcsc.com/szlcsc/1811141223_TOGIALED-TJ-S1608SW6TGLC2G-A5_C192316.pdf" H 1850 3700 50  0001 C CNN
@@
 P 2050 3700
 F 0 "D2" V 2100 3600 50  0000 R CNN
-F 1 "LED" V 2000 3600 50  0000 R CNN
+F 1 "RX" V 2000 3600 50  0000 R CNN
 F 2 "LED_SMD:LED_0805_2012Metric_Pad1.15x1.40mm_HandSolder" H 2050 3700 50  0001 C CNN
 F 3 "https://datasheet.lcsc.com/szlcsc/1811141223_TOGIALED-TJ-S1608SW6TGLC2G-A5_C192316.pdf" H 2050 3700 50  0001 C CNN
@@
 P 900 1850
 F 0 "J4" H 818 1525 50  0000 C CNN
-F 1 "Screw_Terminal_01x02" H 750 1600 50  0000 C CNN
+F 1 "DC 5.5 - 42V" H 750 1600 50  0000 C CNN
 F 2 "TerminalBlock:TerminalBlock_bornier-2_P5.08mm" H 900 1850 50  0001 C CNN
 F 3 "https://datasheet.lcsc.com/szlcsc/1912251632_Ningbo-Kangnex-Elec-WJ15EDGRC-3-81-2P_C8387.pdf" H 900 1850 50  0001 C CNN

Commit message: add(hw): labels and 3D models
Changed lines of the file:
@@
 Text Notes 10170 4210 0    50   ~ 0
 Level shifter as\nMCU is 3.3V but\nWS2812B needs 5V
+$Comp
+L Graphic:Logo_Open_Hardware_Small #LOGO1
+U 1 1 5FF1B0E3
+P 10940 6875
+F 0 "#LOGO1" H 10940 7150 50  0001 C CNN
+F 1 "Logo_Open_Hardware_Small" H 10940 6650 50  0001 C CNN
+F 2 "" H 10940 6875 50  0001 C CNN
+F 3 "~" H 10940 6875 50  0001 C CNN
+	1    10940 6875
+	1    0    0    -1
+$EndComp
 $EndSCHEMATC

Commit message: add: new BOM and update *.sch to new symbol lib
Parts:
- C1, C10, C12, C13, C6, C8: symbol Device:CP1 -> blueled-rescue:CP1-Device
- JP1, JP2: symbol Device:Jumper_NC_Small -> blueled-rescue:Jumper_NC_Small-Device
- L1: symbol Device:L_Core_Iron -> blueled-rescue:L_Core_Iron-Device
- U1: symbol MCU_Microchip_ATmega:ATmega328P-AU -> blueled-rescue:ATmega328P-AU-MCU_Microchip_ATmega
Changed lines of the file:
@@
 	2300 5300 2450 5300
 $Comp
-L Device:Jumper_NC_Small JP1
+L blueled-rescue:Jumper_NC_Small-Device JP1
 U 1 1 5EA9BCB4
 P 2250 4200
@@
 $EndComp
 $Comp
-L Device:Jumper_NC_Small JP2
+L blueled-rescue:Jumper_NC_Small-Device JP2
 U 1 1 5EAABDED
 P 2250 4300
@@
 LED strip & MCU \n     POWER
 $Comp
-L Device:CP1 C12
+L blueled-rescue:CP1-Device C12
 U 1 1 6068EAC3
 P 5800 4250
@@
 XY2500F-B-5.08-3P \nfor LED strip\n
 $Comp
-L Device:CP1 C6
+L blueled-rescue:CP1-Device C6
 U 1 1 5FD6E875
 P 1625 1250
@@
 	6000 1550 6275 1550
 $Comp
-L Device:CP1 C13
+L blueled-rescue:CP1-Device C13
 U 1 1 5FEE1E45
 P 6275 1725
@@
 	4200 2550 4750 2550
 $Comp
-L Device:CP1 C1
+L blueled-rescue:CP1-Device C1
 U 1 1 5EA4B8BA
 P 3650 2300
@@
 $EndComp
 $Comp
-L Device:CP1 C8
+L blueled-rescue:CP1-Device C8
 U 1 1 5FE6F1B7
 P 3450 850
@@
 $EndComp
 $Comp
-L Device:CP1 C10
+L blueled-rescue:CP1-Device C10
 U 1 1 5FE853F6
 P 6000 1725
@@
 $EndComp
 $Comp
-L Device:L_Core_Iron L1
+L blueled-rescue:L_Core_Iron-Device L1
 U 1 1 5FE6D6CD
 P 5000 1200
@@
 $EndComp
 $Comp
-L MCU_Microchip_ATmega:ATmega328P-AU U1
+L blueled-rescue:ATmega328P-AU-MCU_Microchip_ATmega U1
 U 1 1 5CAE668A
 P 8250 2650
